File: oroca_bldc_SCH/design/OROCA_BLDC.sch (KiCad schematic (older format))
At the start: 48 parts, among them U2 TC2117, U3 DRV8302

Commit message: - kicad를 이용하여 회로도 작성(최종상태 반영) - 아트웍 작업 필요
Parts:
- removed C25, C33: 100u, w_smd_cap:c_tant_B, symbol CP1-RESCUE-BLDC_4
- removed C28: 220n, CRF1:SMD-0603_c, symbol C-RESCUE-BLDC_4
- removed U2: TC2117, CRF1:SOT-223, symbol NCP1117ST33T3G
- removed U3: DRV8302, CRF1:TSSOP-56-PP, symbol DRV8302
- added A1: MOTOR3, CRF1:1PAD_4x5mm, symbol CONN_1
- added B1: MOTOR2, CRF1:1PAD_4x5mm, symbol CONN_1
- added C10, C5, C7: 4n7, CRF1:SMD-0603_c, symbol C-RESCUE-BLDC_4
- added C11, C17: 15p, CRF1:SMD-0603_c, symbol C-RESCUE-BLDC_4
- added C12, C13, C14, C16, C2, C3, C32, C33, C4, C6: 2.2u, CRF1:SMD-0603_c, symbol C-RESCUE-BLDC_4
- added C15: 100n, CRF1:SMD-0603_c, symbol C-RESCUE-BLDC_4
- added C25: 6.8n, CRF1:SMD-0603_c, symbol C-RESCUE-BLDC_4
- added C28, C48: 100u, w_smd_cap:c_tant_B, symbol CP1-RESCUE-BLDC_4
- added C31: 22n, CRF1:SMD-0603_c, symbol C-RESCUE-BLDC_4
- added C35, C45, C46, C47, C50: 10u,50V, CRF1:SMD-1206, symbol C-RESCUE-BLDC_4
- added C38: 15n, CRF1:SMD-0603_c, symbol C-RESCUE-BLDC_4
- added C41, C42: 220n, CRF1:SMD-0603_c, symbol C-RESCUE-BLDC_4
- added C53: MOTOR1, CRF1:1PAD_4x5mm, symbol CONN_1
- added D1: GREEN, LEDs:LED-0603, symbol LED-RESCUE-BLDC_4
- added D2: RED, LEDs:LED-0603, symbol LED-RESCUE-BLDC_4
- added D3: LED, LEDs:LED-0603, symbol LED-RESCUE-BLDC_4
- added J1, J10, J11, J12, J13, J14, J2, J3, J4, J5, J6, J7, J8, J9: TP, Wire_Pads:SolderWirePad_single_0-8mmDrill, symbol TEST_1P
- added K1: SERVO, CRF1:pinhead-1X03, symbol CONN_3
- added P1: PWR_COMM, CRF1:b7b-ph-kl, symbol CONN_01X07
- added P2: AHALL/BEMF, CRF1:MICRO_JST_6, symbol CONN_6
- added P3: CANBUS, JST conn:b4b-ph-kl, symbol CONN_4
- added P4: SWD, CRF1:MICRO_JST_6, symbol CONN_6
- added P5: DHALL/ENC, CRF1:MICRO_JST_6, symbol CONN_6
- added P6: IN+, CRF1:1PAD_4x5mm, symbol CONN_1
- added P7: IN-, CRF1:1PAD_4x5mm, symbol CONN_1
- added Q1: 2N7002, TO_SOT_Packages_SMD:SOT-23, symbol 2N7002
- added Q2, Q3, Q4, Q5, Q6, Q7: IRFS7530, CRF1:D2PAK-7-GDS, symbol MOSFET_N
- added R1, R31: 0R, CRF1:SMD-0603_r, symbol R-RESCUE-BLDC_4
- added R10, R14, R29, R7, R8, R9: 10k, CRF1:SMD-0603_r, symbol R-RESCUE-BLDC_4
- added R11, R12, R13, R15, R22, R38, R53: 2k2, CRF1:SMD-0603_r, symbol R-RESCUE-BLDC_4
- added R16: 4.7k, CRF1:SMD-0603_r, symbol R-RESCUE-BLDC_4
- added R2, R3: 22R, CRF1:SMD-0603_r, symbol R-RESCUE-BLDC_4
- added R28: 220k, CRF1:SMD-0603_r, symbol R-RESCUE-BLDC_4
- added R30, R54, R55, R56: NC, CRF1:SMD-0603_r, symbol R-RESCUE-BLDC_4
- added R34, R35, R45, R46, R57, R58: 4R7, CRF1:SMD-0603_r, symbol R-RESCUE-BLDC_4
- added R36, R37, R47, R52, R59: 39k, CRF1:SMD-0603_r, symbol R-RESCUE-BLDC_4
- added R39, R60: SHUNT, CRF1:WSLP2726, symbol SHUNT
- added R4, R41, R42, R43, R44, R5: 100R, CRF1:SMD-0603_r, symbol R-RESCUE-BLDC_4
- added R40: 1M, CRF1:SMD-0603_r, symbol R-RESCUE-BLDC_4
- added R6: NI, CRF1:SMD-0603_r, symbol R-RESCUE-BLDC_4
- added U1: STM32F40X_LQFP64, CRF1:lqfp64_pad_mod, symbol STM32F40X_LQFP64
- added U2: SN65HVD232, CRF1:SOIC-8-W, symbol MCP2551-I/SN-RESCUE-BLDC_4
- added U3: TC2117, CRF1:SOT-223, symbol NCP1117ST33T3G
- added U4: DRV8302, CRF1:TSSOP-56-PP, symbol DRV8302
- added X1: MINI-USB-SHIELD-32005-201, CRF1:USB-UX60R-MB-5ST, symbol MINI-USB-SCHIELD-32005-201
- added Y1: 8Mhz,10ppm, ABM3B-8.0-10-1UT, symbol Crystal_GND3
- C1, C9: value 10u,50V -> 2.2u; footprint CRF1:SMD-1206 -> CRF1:SMD-0603_c
- C18: value 2.2u -> 100n
- C19: value 120p -> 4n7
- C20, C23: value 2.2u -> 4n7
- C21: value 6.8n -> 4n7
- C22: value 22n -> 2.2u
- C26: value 2.2u -> 120p
- C27: value 100n -> 2.2u
- C29, C30: value 220n -> 2.2u
- C34, C36: value 2.2n -> 10u,50V; footprint CRF1:SMD-0603_c -> CRF1:SMD-1206
- C37: value 15u,100V -> 100n; footprint w_smd_cap:c_2220 -> CRF1:SMD-0603_c
- C39: value 10u,50V -> 100n; footprint CRF1:SMD-1206 -> CRF1:SMD-0603_c
- C40: value 10u,50V -> 220n; footprint CRF1:SMD-1206 -> CRF1:SMD-0603_c
- C43, C44: value 10u,50V -> 2.2n; footprint CRF1:SMD-1206 -> CRF1:SMD-0603_c
- C49: value 10u,50V -> 15u, 100v; footprint CRF1:SMD-1206 -> w_smd_cap:c_2220
- C51: value 15u, 100v -> 10u,50V; footprint w_smd_cap:c_2220 -> CRF1:SMD-1206
- C52: value 2.2u -> 15u,100V; footprint CRF1:SMD-0603_c -> w_smd_cap:c_2220
- C8: value 10u,50V -> 4n7; footprint CRF1:SMD-1206 -> CRF1:SMD-0603_c
- R17: value 18k -> 10k
- R18: value 3k3 -> 10k
- R19: value 15k -> 10k
- R21: value 220k -> 4.7k
- R23, R26: value 39k -> 2k2
- R24: value 2k2 -> 18k
- R25: value 1M -> 3k3
- R27: value 2k2 -> 15k
- R32: value 39k -> NTC 10k
- R33: value 2k2 -> 10k
- R48, R50: value 100R -> 39k
- R49, R51: value 100R -> 2k2
Connections:
- net labels added: AN_IN, CAN_RX, CAN_TX, ENC1/DHALL1, ENC2/DHALL2, ENC3/DHALL3, GND-RESCUE-BLDC_4, INV_TEMP, MISO_ADC_EXT2, MOTOR_TEMP1, MOTOR_TEMP2, NRST, RX_SCL_MOSI, SCK_ADC_EXT, SERVO, SWCLK, SWDIO, TX_SDA_NSS, USB_DM, USB_DP
- wire segments 189 -> 367
- no-connect marks 4 -> 3
Other:
- note added: "Bypass, place next to VDD pins"
- note added: "ESD protection?\n"
- note added: "Mount 0R if used\nas USB host"
- note added: "Programming / Debug\nconnector"
- note added: "Propagation delay\nresistor"
- note added: "Required for USB\nto work"
- note added: "Reset pin internally\npulled up"
- note added: "Voltage supply (0 - 60v)\nNeeds external decoupling\ncaps to avoid high voltage\ntransients produced by the\ninductance of the battery\nwiring while switching the FETs\nAlso critical for EMI/RF compliance"
- note removed: "MCU must sense the\nvoltage at each phase"
